File: Design.kicad_sch (KiCad schematic)
At the start: 8 parts, among them U1 TP4056

Commit message: Add files via upload
Parts:
- added C1, C6: C_Polarized_US, symbol Device:C_Polarized_US
- added C2, C3, C4, C5, C7, C8: C, symbol Device:C
- added D1: D_Zener, symbol Device:D_Zener
- added J2, J3: Conn_01x01_Pin, symbol Connector:Conn_01x01_Pin
- added J4: Conn_01x02_Pin, symbol Connector:Conn_01x02_Pin
- added L1: L, symbol Device:L
- added R1: R_Shunt, symbol Device:R_Shunt
- added R2, R3: R, symbol Device:R
- added U1: TPS54331DR, DESIGN:SOIC-8_L5.0-W4.0-P1.27-LS6.0-BL, symbol SCHLIB_TPS54331DR_2025-03-24:TPS54331DR
- added U2: INA219AIDCNR, symbol SCHLIB_INA219AIDCNR_2025-03-24:INA219AIDCNR
- added currentlim1, currentlim2, currentlim3, currentlim4, currentlim5: R_Small_US, symbol Device:R_Small_US
- renumbered D2 to D?, R2 to R?
Connections:
- net 5V Reg: now also C6.1, L1.2, currentlim1.1
- net GND: now also R1.2, U1.1 (TEMP), C1.2, C3.1, C4.1, C6.2, C7.2, C8.1, C8.2, D1.2 (A), R1.4, U1.7 (GND), U2.3 (GND), currentlim2.2, currentlim4.1, currentlim5.2
- new net: U1.5 (VSENSE), currentlim1.2, currentlim2.1
- new net: C5.1, currentlim5.1
- new net: C4.2, C5.2, U1.6 (COMP)
- new net: U1.3 (EN), currentlim3.2, currentlim4.2
- new net: C2.1, D1.1 (K), L1.1, U1.8 (PH)
- new net: C2.2, U1.1 (BOOT)
- new net: C3.2, U1.4 (SS)
- new net BAT+: J4.1 (Pin_1), U2.1 (IN+)
- new net BAT-: J4.2 (Pin_2), R1.2, U2.2 (IN-)
- new net PB8: J3.1 (Pin_1), R2.2, U2.5 (SCL)
- new net PB9: J2.1 (Pin_1), R3.2, U2.6 (SDA)
- new net VCC: C1.1, U1.2 (VIN), currentlim3.1
- new net VCC -uC: C7.1, R2.1, R3.1, U2.4 (VS)

Commit message: Add files via upload
Parts:
- removed U1: TP4056, KICAD:ESOP-8_L4.9-W3.9-P1.27-LS6.0-BL-EP, symbol SCHLIB_TP4056_2025-03-23:TP4056
- removed U1: TPS54331DR, DESIGN:SOIC-8_L5.0-W4.0-P1.27-LS6.0-BL, symbol SCHLIB_TPS54331DR_2025-03-24:TPS54331DR
- added J1: Conn_02x16_Odd_Even, Connector_PinSocket_2.54mm:PinSocket_2x16_P2.54mm_Vertical_SMD, symbol Connector_Generic:Conn_02x16_Odd_Even
- added J5: Conn_01x02, Connector_JST:JST_PH_S2B-PH-K_1x02_P2.00mm_Horizontal, symbol Connector_Generic:Conn_01x02
- added Q1: DMP3099L, PCM_JLCPCB:SOT-23-3_L2.9-W1.3-P0.95-LS2.4-BR, symbol Transistor_FET:DMP3099L
- added Q2: 2N7002, PCM_JLCPCB:Q_SOT-23, symbol PCM_JLCPCB-Transistors:NMOS,2N7002
- added Q3: SI2301CDS-T1-GE3, PCM_JLCPCB:Q_SOT-23, symbol PCM_JLCPCB-Transistors:PMOS,SI2301CDS-T1-GE3
- added U1: AMS1117, PCM_JLCPCB:SOT-223-3_L6.5-W3.4-P2.30-LS7.0-BR, symbol PCM_JLCPCB-Power:LDO, 3.3V, 1A
- added U3: TP4056, PCM_JLCPCB:ESOP-8_L4.9-W3.9-P1.27-LS6.0-BL-EP, symbol PCM_JLCPCB-Power:Battery, Li-Ion, 1.0A, TP4056
- added U4: TPS54331DR, PCM_JLCPCB:SOIC-8_L5.0-W4.0-P1.27-LS6.0-BL, symbol PCM_JLCPCB-Power:DC-DC, Buck, 3.5-28VIN, 3A, 0.8+VOUT
- added U5: DRV8833PWP, Package_SO:HTSSOP-16-1EP_4.4x5mm_P0.65mm_EP3.4x5mm_Mask2.46x2.31mm_ThermalVias, symbol Driver_Motor:DRV8833PWP
- added U6: MT3608L, symbol SCHLIB_MT3608L_2025-03-27:MT3608L
- added U7: TPS54331DR, symbol SCHLIB_TPS54331DR_2025-03-24:TPS54331DR
- added USB1: TYPE-C 16PIN 2MD(073), symbol SCHLIB_TYPE-C-16PIN-2MD(073)_2025-03-27:TYPE-C 16PIN 2MD(073)
- gave numbers to parts that had none: 2
- renumbered C2 to C10, C1 to C9, D1 to D3, R1 to R5, currentlim to currentlim6
Connections:
- net 5V Reg: now also U3.4 (VCC); no longer C6.1, L1.2, currentlim1.1
- net Bat+Protection IC: now also U3.5 (BAT)
- net GND: now also J1.19 (Pin_19), J1.23 (Pin_23), U3.1 (TEMP), U3.3 (GND), U3.9 (EP), U4.7 (GND)
- net GPIO pin: now also U3.8 (CE)
- net VCC: now also U4.2 (VIN)
- net at R4.2: now also U3.7 (CHRG#)
- net VSENSE: now reaches currentlim1.2, currentlim2.1
- net VSENSE: now also U4.5 (VSENSE)
- net COMP: now reaches C4.2, C5.2
- net COMP: now also U4.6 (COMP)
- net EN: now reaches currentlim3.2, currentlim4.2
- net EN: now also U4.3 (EN)
- net at R5.1: now also U3.2 (PROG)
- net at currentlim6.2: now also U3.6 (STDBY#)
- net PH: now reaches C2.1, D1.1 (K), L1.1
- net PH: now also U4.8 (PH)
- net BOOT: now reaches C2.2
- net BOOT: now also U4.1 (BOOT)
- net SS: now reaches C3.2
- net SS: now also U4.4 (SS)
- new net: U5.13 (GND), U5.17 (GND)
- new net: C6.1, L1.2, currentlim1.1
- new net: U1.2 (VOUT), U1.4 (VOUT)
- new net 3V3 Out : J1.18 (Pin_18)
- new net 5V Out : J1.20 (Pin_20)
- new net Battery : J1.14 (Pin_14)
- new net CTRL_EXT_LOAD1: J1.25 (Pin_25)
- new net CTRL_EXT_LOAD2 : J1.7 (Pin_7)
- new net EXT_LOAD1_OUT: J1.21 (Pin_21)
- new net EXT_LOAD2_OUT : J1.11 (Pin_11)
- new net FAST_CHARGE_CTRL: J1.13 (Pin_13)
- new net High Voltage (9V): J1.22 (Pin_22)
- new net I2C1_SCL: J1.16 (Pin_16)
- new net I2C1_SDA : J1.15 (Pin_15)
- new net MOTOR1_A_OUT: J1.32 (Pin_32)
- new net MOTOR1_B_OUT : J1.31 (Pin_31)
- new net MOTOR1_CTRL1: J1.28 (Pin_28)
- new net MOTOR1_CTRL2: J1.30 (Pin_30)
- new net MOTOR2_CTRL1: J1.4 (Pin_4)
- new net MOTOR2_CTRL2: J1.6 (Pin_6)
- new net MOTOR3_A_OUT: J1.27 (Pin_27)
- new net MOTOR3_B_OUT: J1.29 (Pin_29)
- new net MOTOR3_CTRL1: J1.24 (Pin_24)
- new net MOTOR3_CTRL2: J1.26 (Pin_26)
- new net MOTOR4_CTRL1: J1.8 (Pin_8)
- new net MOTOR4_CTRL2: J1.10 (Pin_10)
- new net Motor2_A_OUT : J1.2 (Pin_2)
- new net Motor2_B_OUT: J1.1 (Pin_1)
- new net Motor4_A_OUT : J1.3 (Pin_3)
- new net Motor4_B_OUT: J1.5 (Pin_5)
- new net USART2_RX: J1.9 (Pin_9)
- new net USART2_TX : J1.12 (Pin_12)
- no-connect marks 0 -> 1
Other:
- note added: "Battery Charging System"
- note added: "Power Monitoring"
- note added: "Voltage Regulation (9V to 5V)"
- moved on the sheet: C1, C10, C2, C3, C4, C5, C6, C7, C8, C9, D1, D2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

Commit message: Add files via upload
Parts:
- removed C1, C6: C_Polarized_US, symbol Device:C_Polarized_US
- removed C10, C2, C3, C4, C5, C7, C8, C9: C, symbol Device:C
- removed D1: D_Zener, symbol Device:D_Zener
- removed D2, D3: SFH4346, LED_THT:LED_D3.0mm_IRBlack, symbol LED:SFH4346
- removed J2, J3: Conn_01x01_Pin, symbol Connector:Conn_01x01_Pin
- removed J4: Conn_01x02_Pin, symbol Connector:Conn_01x02_Pin
- removed L1: L, symbol Device:L
- removed R1: R_Shunt, symbol Device:R_Shunt
- removed R2, R3: R, symbol Device:R
- removed R4, R5, currentlim1, currentlim2, currentlim3, currentlim4, currentlim5, currentlim6: R_Small_US, symbol Device:R_Small_US
- removed U7: TPS54331DR, symbol SCHLIB_TPS54331DR_2025-03-24:TPS54331DR
- added C1, C4, C5, C7: 10uF, PCM_JLCPCB:C_0603, symbol PCM_JLCPCB-Capacitors:0603,10uF
- added C10, C17, C18, C19, C20, C8: 100nF, PCM_JLCPCB:C_0402, symbol PCM_JLCPCB-Capacitors:0402,100nF
- added C11, C15, C2, C6, C9: 22uF, PCM_JLCPCB:C_0603, symbol PCM_JLCPCB-Capacitors:0603,22uF
- added C12, C16: 10uF, PCM_JLCPCB:C_0805, symbol PCM_JLCPCB-Capacitors:0805,10uF
- added C13, C14, C3: 10nF, PCM_JLCPCB:C_0402, symbol PCM_JLCPCB-Capacitors:0402,10nF
- added D1: Red, PCM_JLCPCB:D_0603, symbol PCM_JLCPCB-Diodes:LED,0603,Red
- added D4, D6, D7: 1N4148WS, PCM_JLCPCB:D_SOD-323, symbol PCM_JLCPCB-Diodes:Switching,1N4148WS
- added D5, D8: White, PCM_JLCPCB:D_0603, symbol PCM_JLCPCB-Diodes:LED,0603,White
- added L1: 10uH,25mA, PCM_JLCPCB:L_1206, symbol PCM_JLCPCB-Inductors:10uH,25mA
- added L3: 4.7uH,15mA, PCM_JLCPCB:L_0603, symbol PCM_JLCPCB-Inductors:4.7uH,15mA
- added Q4, Q5: DMP3099L, PCM_JLCPCB:SOT-23-3_L2.9-W1.3-P0.95-LS2.4-BR, symbol Transistor_FET:DMP3099L
- added R1: 1Ω, PCM_JLCPCB:R_0603, symbol PCM_JLCPCB-Resistors:0603,1Ω
- added R10, R14, R4: 1kΩ, PCM_JLCPCB:R_0402, symbol PCM_JLCPCB-Resistors:0402,1kΩ
- added R11, R15, R6, R9: 100kΩ, PCM_JLCPCB:R_0603, symbol PCM_JLCPCB-Resistors:0603,100kΩ
- added R12: 120kΩ, PCM_JLCPCB:R_0402, symbol PCM_JLCPCB-Resistors:0402,120kΩ
- added R13, R5: 5.1kΩ, PCM_JLCPCB:R_0402, symbol PCM_JLCPCB-Resistors:0402,5.1kΩ
- added R16: 8.2kΩ, PCM_JLCPCB:R_0402, symbol PCM_JLCPCB-Resistors:0402,8.2kΩ
- added R2, R3: 4.7kΩ, PCM_JLCPCB:R_0402, symbol PCM_JLCPCB-Resistors:0402,4.7kΩ
- added R7: 10kΩ, PCM_JLCPCB:R_0402, symbol PCM_JLCPCB-Resistors:0402,10kΩ
- added R8: 33kΩ, PCM_JLCPCB:R_0402, symbol PCM_JLCPCB-Resistors:0402,33kΩ
- added SW1: SW_SPDT, symbol Switch:SW_SPDT
- added U8: DRV8833PWP, Package_SO:HTSSOP-16-1EP_4.4x5mm_P0.65mm_EP3.4x5mm_Mask2.46x2.31mm_ThermalVias, symbol Driver_Motor:DRV8833PWP
- Q1: Part (none) -> C2940610
Connections:
- net Bat+Protection IC is gone; now on net BAT+: U3.5 (BAT)
- net COMP is gone; now on net GND: U4.6 (COMP)
- net EN is gone; now on net VCC: U4.3 (EN)
- net PB8 is gone; now on net I2C1_SCL: U2.5 (SCL)
- net PB9 is gone; now on net I2C1_SDA : U2.6 (SDA)
- net SS is gone; now on net GND: U4.4 (SS)
- net VCC -uC is gone; now on net 3V3 Out : U2.4 (VS)
- net 3V3 Out : now also Q2.1 (G), C7.1, R2.2, R3.2
- net BAT+: now also J5.2 (Pin_2), C5.2
- net BAT-: now also J5.1 (Pin_1), R1.2
- net Battery : now also SW1.1 (A)
- net GND: now also Q1.2 (S), Q2.2 (S), U1.1 (GND), U5.13 (GND), U5.17 (GND), U5.3 (AISEN), U5.6 (BISEN), U6.2 (GND), USB1.1 (GND), USB1.12 (GND), C1.1, C10.2, C11.1, C13.1, C14.1, C15.1, C17.2, C18.2, C19.2, C2.2, C4.1, C5.1, C7.2, C8.2, D4.1, D6.1, D7.1, D8.1, Q4.2 (S), Q5.2 (S), R1.1, R13.1, R15.2, R16.1, R5.1, R7.2, U8.13 (GND), U8.17 (GND), U8.3 (AISEN), U8.6 (BISEN); no longer U2.3 (GND)
- net GPIO pin: now also R6.1, R9.1; no longer U3.8 (CE)
- net I2C1_SCL: now also R2.1
- net I2C1_SDA : now also R3.1
- net Motor2_A_OUT : now also U5.2 (AOUT1)
- net Motor2_B_OUT: now also U5.4 (AOUT2)
- net Motor4_A_OUT : now also U5.7 (BOUT1)
- net Motor4_B_OUT: now also U5.5 (BOUT2)
- net VCC: now also C1.2
- net at Q3.1 (G): now also Q2.3 (D), C10.1, R15.1
- net at Q3.2 (S): now also SW1.2 (B)
- net at Q3.3 (D): now also C20.1
- net 3.3 V: now reaches U5.1 (~{SLEEP})
- net 3.3 V: now also U1.2 (VOUT), U1.4 (VOUT), U8.1 (~{SLEEP})
- net PD15: now reaches U5.10 (BIN2)
- net at U5.11 (VCP): now also C13.2
- net at U5.12 (VM): now also C12.1
- net at U5.14 (VINT): now also C11.2
- net PD13: now reaches U5.15 (AIN2)
- net PD12: now reaches U5.16 (AIN1)
- net PD14: now reaches U5.9 (BIN1)
- net at U3.7 (CHRG#): now also R4.2
- net at USB1.10 (CC2): now also R13.2
- net at USB1.11 (VBUS): now also USB1.2 (VBUS), C9.1
- net at USB1.4 (CC1): now also R5.2
- net at U3.6 (STDBY#): now also R10.2
- net at U3.2 (PROG): now also R11.1
- net at Q1.1 (G): now also C17.1, R6.2
- net at Q1.3 (D): now also D4.2
- net 9V input: now reaches U1.3 (VIN)
- net at U6.1 (SW): now also L3.2
- net at U6.3 (FB): now also R12.2, R16.2
- net at U6.4 (EN): now also U6.5 (VIN), C9.2
- net 5V Reg renamed 5V 
- net 5V : now also U3.8 (CE), C4.2, D1.2, D5.2
- net BOOT: no longer names the net of U4.1 (BOOT)
- net BOOT: now also C3.1
- net PH: no longer names the net of U4.8 (PH)
- net PH: now also C3.2, L1.1
- net VSENSE: no longer names the net of U4.5 (VSENSE)
- net VSENSE: now also R7.1, R8.2
- new net: C18.1, Q4.1 (G), R9.2
- new net: D7.2, Q5.3 (D)
- new net: C16.1, U8.12 (VM)
- new net: C19.1, Q5.1 (G), R11.2
- new net: C8.1, U2.3 (GND)
- new net: C6.1, R12.1
- new net: C6.2, L3.1
- new net: D1.1, R4.1
- new net: R14.1, SW1.3 (C)
- new net: C14.2, U8.11 (VCP)
- new net: D8.2, R14.2
- new net: C15.2, U8.14 (VINT)
- new net: D5.1, R10.1
- new net: D6.2, Q4.3 (D)
- new net 5 V: C2.1, C20.2, L1.2, R8.1
- new net Bat+: C12.2, C16.2
- new net MOTOR1_B_OUT: U8.5 (BOUT2)
- new net Motor1_A_OUT : U8.7 (BOUT1)
- new net Motor3_B_OUT: U8.4 (AOUT2)
- new net PC6: U8.9 (BIN1)
- new net PC7: U8.10 (BIN2)
- new net PC8: U8.16 (AIN1)
- new net PC9: U8.15 (AIN2)
- new net PCP: U8.2 (AOUT1)
- no-connect marks 1 -> 4
Other:
- note added: "Motor Control Auxiliary motors"
- note added: "Motor Control Mains motors"
- moved on the sheet: J1, J5, Q1, Q2, Q3, U1, U2, U3, U4, U5, U6, USB1

Commit message: Add files via upload
Parts:
- removed D7: 1N4148WS, PCM_JLCPCB:D_SOD-323, symbol PCM_JLCPCB-Diodes:Switching,1N4148WS
- removed R11: 100kΩ, PCM_JLCPCB:R_0603, symbol PCM_JLCPCB-Resistors:0603,100kΩ
- added R11: 5.1kΩ, PCM_JLCPCB:R_0402, symbol PCM_JLCPCB-Resistors:0402,5.1kΩ
- added R17: 2.2kΩ, PCM_JLCPCB:R_0402, symbol PCM_JLCPCB-Resistors:0402,2.2kΩ
- added R18: 100kΩ, PCM_JLCPCB:R_0603, symbol PCM_JLCPCB-Resistors:0603,100kΩ
- added TP1, TP10, TP11, TP12, TP13, TP14, TP15, TP16, TP17, TP18, TP19, TP2, TP20, TP21, TP22, TP23, TP24, TP25, TP26, TP27, TP3, TP4, TP5, TP6, TP7, TP8, TP9: TestPoint, symbol Connector:TestPoint
Connections:
- net 3.3 V is gone; now on net 3V3 Out : U1.2 (VOUT), U1.4 (VOUT), U5.1 (~{SLEEP}), U8.1 (~{SLEEP})
- net 5 V is gone; now on net 5V Out : C2.1, C20.2, L1.2, R8.1
- net 9V input is gone; now on net High Voltage (9V): U1.3 (VIN)
- net Bat+ is gone; now on net GND: C12.2, C16.2
- net Battery  is gone; now on net BAT+: J1.14 (Pin_14), SW1.1 (A)
- net MOTOR1_B_OUT is gone; now on net Motor4_B_OUT: U8.5 (BOUT2)
- net Motor1_A_OUT  is gone; now on net MOTOR3_B_OUT: U8.7 (BOUT1)
- net Motor3_B_OUT is gone; now on net Motor4_A_OUT : U8.4 (AOUT2)
- net PC6 is gone; now on net MOTOR3_CTRL1: U8.9 (BIN1)
- net PC7 is gone; now on net MOTOR3_CTRL2: U8.10 (BIN2)
- net PC8 is gone; now on net MOTOR4_CTRL1: U8.16 (AIN1)
- net PC9 is gone; now on net MOTOR4_CTRL2: U8.15 (AIN2)
- net PCP is gone; now on net MOTOR3_A_OUT: U8.2 (AOUT1)
- net PD12 is gone; now on net MOTOR2_CTRL1: U5.16 (AIN1)
- net PD13 is gone; now on net MOTOR2_CTRL2: U5.15 (AIN2)
- net PD14 is gone; now on net MOTOR1_CTRL1: U5.9 (BIN1)
- net PD15 is gone; now on net MOTOR1_CTRL2: U5.10 (BIN2)
- net VCC is gone; now on net High Voltage (9V): C1.2, U4.2 (VIN), U4.3 (EN)
- net 3V3 Out : now also TP19.1
- net 5V Out : now also TP23.1
- net BAT+: now also C12.1, C16.1, U5.12 (VM), U8.12 (VM)
- net BAT-: now also TP21.1
- net CTRL_EXT_LOAD1: now also R9.1, TP4.1
- net CTRL_EXT_LOAD2 : now also R6.1, TP6.1
- net EXT_LOAD1_OUT: now also D6.2, Q4.3 (D)
- net EXT_LOAD2_OUT : now also D4.2, Q1.3 (D)
- net FAST_CHARGE_CTRL: now also R18.1, TP9.1
- net GND: now also R17.2, TP13.1, TP15.1, TP22.1, TP24.1, TP3.1, TP8.1
- net High Voltage (9V): now also C6.1, R12.1, TP11.1
- net I2C1_SCL: now also TP20.1
- net I2C1_SDA : now also TP18.1
- net MOTOR1_A_OUT: now also U5.7 (BOUT1)
- net MOTOR1_B_OUT : now also U5.5 (BOUT2)
- net Motor4_A_OUT : no longer U5.7 (BOUT1)
- net Motor4_B_OUT: no longer U5.5 (BOUT2)
- net at C10.1, Q2.3 (D), Q3.1 (G)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: now also TP14.1
- net at C17.1, Q1.1 (G), R6.2: now also TP7.1
- net at C18.1, Q4.1 (G), R9.2: now also TP5.1
- net at Q5.3 (D): now also R11.2, TP1.1
- net at R13.2, USB1.10 (CC2): now also TP27.1
- net at R5.2, USB1.4 (CC1): now also TP26.1
- net PROG: now reaches U3.2 (PROG)
- net PROG: now also R11.1, R17.1, TP2.1
- net at C19.1, Q5.1 (G): now also R18.2, TP10.1
- net at R12.2, R16.2, U6.3 (FB): now also TP12.1
- net at R14.1, SW1.3 (C): now also TP16.1
- net at D8.2, R14.2: now also TP17.1
- net at R7.1, R8.2, U4.5 (VSENSE): now also TP25.1
- net 5V  renamed 5V Out
- removed net GPIO pin: R6.1, R9.1
- no-connect marks 4 -> 14
Other:
- moved on the sheet: C1, C10, C15, C17, C18, C2, C20, C3, C4, C5, C6, C7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

Commit message: Add files via upload
Parts:
- removed SW1: SW_SPDT, symbol Switch:SW_SPDT
- added SW2: K3-1391B-51, symbol SCHLIB_Switch_K3-1391B-51_2025-04-07:K3-1391B-51
- U2: footprint (none) -> DESIGN:INA219AIDCNR_SOT-23-8_L3.0-W1.7-P0.65-LS2.8-BR
- U6: footprint (none) -> DESIGN:MT3608L_SOT-23-8_L3.0-W1.7-P0.65-LS2.8-BR
- USB1: footprint (none) -> DESIGN:USB-C-SMD_TYPE-C-6PIN-2MD-073
Connections:
- net BAT+: now also SW2.1
- net at Q3.2 (S): now also SW2.2
- net at R14.1, TP16.1: now also SW2.3
- no-connect marks 14 -> 15
Other:
- note added: "Charging Current Programing System"
- note added: "External Load Switching"
- note added: "Motor Control"
- note added: "Power Switch"
- note added: "USB C power"
- note added: "Voltage Regulation (9 V to 3.3 V)"

Commit message: Add files via upload
Parts:
- SW2: footprint (none) -> DESIGN:SW-TH_K3-1391B-51
- TP1, TP10, TP11, TP12, TP13, TP14, TP15, TP16, TP17, TP18, TP19, TP2, TP20, TP21, TP22, TP23, TP24, TP25, TP26, TP27, TP3, TP4, TP5, TP6, TP7, TP8, TP9: footprint (none) -> TestPoint:TestPoint_Pad_D1.0mm
Changed lines of the file:
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@@
 			)
 		)
-		(property "Footprint" ""
+		(property "Footprint" "TestPoint:TestPoint_Pad_D1.0mm"
 			(at 180.34 134.62 0)
 			(effects
@@
 			)
 		)
-		(property "Footprint" ""
+		(property "Footprint" "TestPoint:TestPoint_Pad_D1.0mm"
 			(at 180.34 83.82 0)
 			(effects
@@
 			)
 		)
-		(property "Footprint" ""
+		(property "Footprint" "TestPoint:TestPoint_Pad_D1.0mm"
 			(at 49.53 90.17 0)
 			(effects
@@
 			)
 		)
-		(property "Footprint" ""
+		(property "Footprint" "TestPoint:TestPoint_Pad_D1.0mm"
 			(at 176.53 27.94 0)
 			(effects
@@
 			)
 		)
-		(property "Footprint" ""
+		(property "Footprint" "TestPoint:TestPoint_Pad_D1.0mm"
 			(at 110.49 62.23 0)
 			(effects
@@
 			)
 		)
-		(property "Footprint" ""
+		(property "Footprint" "TestPoint:TestPoint_Pad_D1.0mm"
 			(at 201.93 19.05 0)
 			(effects
@@
 			)
 		)
-		(property "Footprint" ""
+		(property "Footprint" "TestPoint:TestPoint_Pad_D1.0mm"
 			(at 185.42 184.15 0)
 			(effects
@@
 			)
 		)
-		(property "Footprint" ""
+		(property "Footprint" "TestPoint:TestPoint_Pad_D1.0mm"
 			(at 140.97 64.77 0)
 			(effects
@@
 			)
 		)
-		(property "Footprint" ""
+		(property "Footprint" "TestPoint:TestPoint_Pad_D1.0mm"
 			(at 76.2 83.82 0)
 			(effects
@@
 			)
 		)
-		(property "Footprint" ""
+		(property "Footprint" "TestPoint:TestPoint_Pad_D1.0mm"
 			(at 186.69 128.27 0)
 			(effects
@@
 			)
 		)
-		(property "Footprint" ""
+		(property "Footprint" "TestPoint:TestPoint_Pad_D1.0mm"
 			(at 176.53 35.56 0)
 			(effects
@@
 			)
 		)
-		(property "Footprint" ""
+		(property "Footprint" "TestPoint:TestPoint_Pad_D1.0mm"
 			(at 91.44 191.77 0)
 			(effects
@@
 			)
 		)
-		(property "Footprint" ""
+		(property "Footprint" "TestPoint:TestPoint_Pad_D1.0mm"
 			(at 77.47 160.02 0)
 			(effects
@@
 			)
 		)
-		(property "Footprint" ""
+		(property "Footprint" "TestPoint:TestPoint_Pad_D1.0mm"
 			(at 186.69 77.47 0)
 			(effects
@@
 			)
 		)
-		(property "Footprint" ""
+		(property "Footprint" "TestPoint:TestPoint_Pad_D1.0mm"
 			(at 181.61 195.58 0)
 			(effects
@@
 			)
 		)
-		(property "Footprint" ""
+		(property "Footprint" "TestPoint:TestPoint_Pad_D1.0mm"
 			(at 77.47 153.67 0)
 			(effects
@@
 			)
 		)
-		(property "Footprint" ""
+		(property "Footprint" "TestPoint:TestPoint_Pad_D1.0mm"
 			(at 107.95 193.04 0)
 			(effects
@@
 			)
 		)
-		(property "Footprint" ""
+		(property "Footprint" "DESIGN:SW-TH_K3-1391B-51"
 			(at 139.7 43.18 0)
 			(effects
@@
 			)
 		)
-		(property "Footprint" ""
+		(property "Footprint" "TestPoint:TestPoint_Pad_D1.0mm"
 			(at 76.2 105.41 0)
 			(effects
@@
 			)
 		)
-		(property "Footprint" ""
+		(property "Footprint" "TestPoint:TestPoint_Pad_D1.0mm"
 			(at 12.7 134.62 0)
 			(effects
@@
 			)
 		)
-		(property "Footprint" ""
+		(property "Footprint" "TestPoint:TestPoint_Pad_D1.0mm"
 			(at 173.99 16.51 0)
 			(effects
@@
 			)
 		)
-		(property "Footprint" ""
+		(property "Footprint" "TestPoint:TestPoint_Pad_D1.0mm"
 			(at 52.07 148.59 0)
 			(effects
@@
 			)
 		)
-		(property "Footprint" ""
+		(property "Footprint" "TestPoint:TestPoint_Pad_D1.0mm"
 			(at 179.07 190.5 0)
 			(effects
@@
 			)
 		)
-		(property "Footprint" ""
+		(property "Footprint" "TestPoint:TestPoint_Pad_D1.0mm"
 			(at 116.84 55.88 0)
 			(effects
@@
 			)
 		)
-		(property "Footprint" ""
+		(property "Footprint" "TestPoint:TestPoint_Pad_D1.0mm"
 			(at 209.55 41.91 0)
 			(effects
@@
 			)
 		)
-		(property "Footprint" ""
+		(property "Footprint" "TestPoint:TestPoint_Pad_D1.0mm"
 			(at 12.7 140.97 0)
 			(effects
@@
 			)
 		)
-		(property "Footprint" ""
+		(property "Footprint" "TestPoint:TestPoint_Pad_D1.0mm"
 			(at 139.7 55.88 0)
 			(effects
@@
 			)
 		)
-		(property "Footprint" ""
+		(property "Footprint" "TestPoint:TestPoint_Pad_D1.0mm"
 			(at 91.44 182.88 0)
 			(effects
